File: eda/em-lock.kicad_pcb (KiCad board)
At the start: 2 copper layers, 55.9 x 55.9 mm, 78 parts, among them CON1 BARREL_JACK, P1 EXT_LED_CONN, P10 BOOT_SEL_CONN, P12 SWD_CONN, P2 RC522A, P3 RC522B, P4 BTN_OPEN, P5 BTN_CALL, P6 ESP8266_CONN, P7 LOCK_CONN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

Commit message: align with recent develop changes
Parts:
- Q4: value Q_NMOS_DGS -> MOSFET-NCHANNELSMD
- moved H8 11.2 mm to (39.2, 79.1)
- moved H9 7.19 mm to (88.1, 149.6)
- turned Q4 to 180 degrees
Connections:
- P10 pad 1: Net-(P10-Pad1) -> VCC
- P10 pad 2: Net-(P10-Pad1) -> VCC
- Q4 pad 1: LOCK_GND -> Net-(D3-Pad1)
- Q4 pad 2: Net-(D3-Pad1) -> GND
- Q4 pad 3: GND -> LOCK_GND
Routing:
- net GND: track 515.7 -> 502.5 mm
- net VCC: track 476.3 -> 481.4 mm
- net Net-(P10-Pad1): track 2.54 -> 0.00 mm
- net /stm32f103c8/LDO_IN: track 34.0 -> 32.3 mm, vias 2 -> 0
- net LOCK_GND: track 14.9 -> 14.4 mm

Commit message: Revert "Merge branch 'develop'"
This reverts commit ff1c94cd9af79a798b971b643cbdc9d823101f0c, reversing
changes made to 75416340a58c0ce3ae2d4917c1e5600380b4c8a3.
Parts:
- Q4: value MOSFET-NCHANNELSMD -> Q_NMOS_DGS
- moved H8 11.2 mm to (27.9, 78.7)
- moved H9 7.19 mm to (95.2, 149.9)
- turned Q4 to 0 degrees
Connections:
- P10 pad 1: VCC -> Net-(P10-Pad1)
- P10 pad 2: VCC -> Net-(P10-Pad1)
- Q4 pad 1: Net-(D3-Pad1) -> LOCK_GND
- Q4 pad 2: GND -> Net-(D3-Pad1)
- Q4 pad 3: LOCK_GND -> GND
Routing:
- net GND: track 502.5 -> 515.7 mm
- net VCC: track 481.4 -> 476.3 mm
- net Net-(P10-Pad1): track 0.00 -> 2.54 mm
- net /stm32f103c8/LDO_IN: track 32.3 -> 34.0 mm, vias 0 -> 2
- net LOCK_GND: track 14.4 -> 14.9 mm

Commit message: fix problem
Parts:
- moved H8 11.2 mm to (39.2, 79.1)
- moved H9 7.19 mm to (88.1, 149.6)
Routing:
- net GND: track 515.7 -> 512.3 mm
- net /stm32f103c8/LDO_IN: track 34.0 -> 32.3 mm, vias 2 -> 0
