File: eda/em-lock.sch (KiCad schematic (older format))
At the start: 55 parts, among them P1 EXT_LED_CONN, P11 LEDA_CONN, P13 IN_LED_CONN, P14 LEDB_CONN, P15 LEDB_CONN, P2 RC522A, P3 RC522B, P4 BTN_OPEN, P5 BTN_CALL, P6 ESP8266_CONN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

Commit message: refs #41563 pcb done (pochti ;))
Connections:
- net GNDD: now also C21.2, C22.2, P1.4 (P4)
- net GNDREF: no longer C21.2, C22.2, P1.4 (P4)
Changed lines of the file:
@@
 $EndComp
 $Comp
-L GND #PWR05
+L GNDD #PWR05
 U 1 1 582803A4
 P 2800 950
 F 0 "#PWR05" H 2800 700 50  0001 C CNN
-F 1 "GND" V 2800 750 50  0000 C CNN
+F 1 "GNDD" H 2800 800 50  0000 C CNN
 F 2 "" H 2800 950 50  0000 C CNN
 F 3 "" H 2800 950 50  0000 C CNN

Commit message: refs #41563 main pcb done, todo: leds pcb multiplexor
Parts:
- P2: footprint I20:RC522_Full -> I20:b8b-ph-kl
Changed lines of the file:
@@
 	0    1    1    0
 $EndComp
-Text GLabel 8550 3150 0    60   Input ~ 0
-EM_LOCK
 $Comp
 L VDD #PWR04
@@
 F 0 "P2" H 1527 6391 50  0000 L CNN
 F 1 "RC522A" H 1527 6300 50  0000 L CNN
-F 2 "I20:RC522_Full" H 1450 6350 50  0001 C CNN
+F 2 "I20:b8b-ph-kl" H 1450 6350 50  0001 C CNN
 F 3 "" H 1450 6350 50  0000 C CNN
 	1    1450 6350
@@
 Wire Wire Line
 	4800 3650 4800 3900
-Wire Wire Line
-	8550 3150 8950 3150
 Connection ~ 9150 4300
 Wire Wire Line
@@
 	8650 3200 8650 3150
 Connection ~ 8650 3150
-Wire Wire Line
-	8950 3250 8850 3250
 Wire Wire Line
 	8850 3250 8850 3600
@@
 Wire Wire Line
 	2450 3750 2450 3400
+Text GLabel 8550 3150 0    60   Input ~ 0
+EM_LOCK
+Wire Wire Line
+	8550 3150 8950 3150
+Wire Wire Line
+	8850 3250 8950 3250
 $EndSCHEMATC

Commit message: refs #41563 +leds multiplexor + leds pcb's
Parts:
- P11, P13, P14, P15, P8: footprint I20:jst-s4b-ph-kl-angled -> I20:JST_XH_S04B-XH-A_04x2.50mm_Angled
- P2: footprint I20:b8b-ph-kl -> I20:JST_XH_B08B-XH-A_08x2.50mm_Straight
Changed lines of the file:
@@
 F 0 "P2" H 1527 6391 50  0000 L CNN
 F 1 "RC522A" H 1527 6300 50  0000 L CNN
-F 2 "I20:b8b-ph-kl" H 1450 6350 50  0001 C CNN
+F 2 "I20:JST_XH_B08B-XH-A_08x2.50mm_Straight" H 1450 6350 50  0001 C CNN
 F 3 "" H 1450 6350 50  0000 C CNN
 	1    1450 6350
@@
 F 0 "P13" H 2000 4450 50  0000 R CNN
 F 1 "IN_LED_CONN" V 2050 4950 50  0000 R CNN
-F 2 "I20:jst-s4b-ph-kl-angled" H 1950 4700 50  0001 C CNN
+F 2 "I20:JST_XH_S04B-XH-A_04x2.50mm_Angled" H 1950 4700 50  0001 C CNN
 F 3 "" H 1950 4700 50  0000 C CNN
 	1    1950 4700
@@
 F 0 "P8" H 900 3450 50  0000 R CNN
 F 1 "LEDB_CONN" V 950 3950 50  0000 R CNN
-F 2 "I20:jst-s4b-ph-kl-angled" H 850 3700 50  0001 C CNN
+F 2 "I20:JST_XH_S04B-XH-A_04x2.50mm_Angled" H 850 3700 50  0001 C CNN
 F 3 "" H 850 3700 50  0000 C CNN
 	1    850  3700
@@
 F 0 "P11" H 900 4050 50  0000 R CNN
 F 1 "LEDA_CONN" V 950 4550 50  0000 R CNN
-F 2 "I20:jst-s4b-ph-kl-angled" H 850 4300 50  0001 C CNN
+F 2 "I20:JST_XH_S04B-XH-A_04x2.50mm_Angled" H 850 4300 50  0001 C CNN
 F 3 "" H 850 4300 50  0000 C CNN
 	1    850  4300
@@
 F 0 "P15" H 3550 4150 50  0000 R CNN
 F 1 "LEDB_CONN" V 3600 4650 50  0000 R CNN
-F 2 "I20:jst-s4b-ph-kl-angled" H 3500 4400 50  0001 C CNN
+F 2 "I20:JST_XH_S04B-XH-A_04x2.50mm_Angled" H 3500 4400 50  0001 C CNN
 F 3 "" H 3500 4400 50  0000 C CNN
 	1    3500 4400
@@
 F 0 "P14" H 3550 3200 50  0000 R CNN
 F 1 "LEDB_CONN" V 3600 3700 50  0000 R CNN
-F 2 "I20:jst-s4b-ph-kl-angled" H 3500 3450 50  0001 C CNN
+F 2 "I20:JST_XH_S04B-XH-A_04x2.50mm_Angled" H 3500 3450 50  0001 C CNN
 F 3 "" H 3500 3450 50  0000 C CNN
 	1    3500 3450

Commit message: fix PCB before manufacturing
Connections:
- net GNDREF renamed GNDPWR
Changed lines of the file:
@@
 EESchema Schematic File Version 2
+LIBS:em-lock-rescue
 LIBS:power
 LIBS:device
@@
 $EndComp
 $Comp
-L GND #PWR03
-U 1 1 57BF3222
-P 8850 4450
-F 0 "#PWR03" H 8850 4200 50  0001 C CNN
-F 1 "GND" H 8855 4277 50  0000 C CNN
-F 2 "" H 8850 4450 50  0000 C CNN
-F 3 "" H 8850 4450 50  0000 C CNN
-	1    8850 4450
-	1    0    0    -1
-$EndComp
-$Comp
 L ZENER D3
 U 1 1 57BF338B
@@
 $EndComp
 $Comp
-L VDD #PWR04
+L VDD #PWR03
 U 1 1 57BFAAAC
 P 4800 3250
-F 0 "#PWR04" H 4800 3100 50  0001 C CNN
+F 0 "#PWR03" H 4800 3100 50  0001 C CNN
 F 1 "VDD" H 4800 3400 50  0000 C CNN
 F 2 "" H 4800 3250 50  0000 C CNN
@@
 $EndComp
 $Comp
-L GNDD #PWR05
+L GNDD #PWR04
 U 1 1 582803A4
 P 2800 950
-F 0 "#PWR05" H 2800 700 50  0001 C CNN
+F 0 "#PWR04" H 2800 700 50  0001 C CNN
 F 1 "GNDD" H 2800 800 50  0000 C CNN
 F 2 "" H 2800 950 50  0000 C CNN
@@
 $EndComp
 $Comp
-L VDD #PWR06
+L VDD #PWR05
 U 1 1 5829C375
 P 2250 6000
-F 0 "#PWR06" H 2250 5850 50  0001 C CNN
+F 0 "#PWR05" H 2250 5850 50  0001 C CNN
 F 1 "VDD" V 2250 6200 50  0000 C CNN
 F 2 "" H 2250 6000 50  0000 C CNN
@@
 $EndComp
 $Comp
-L GNDD #PWR07
+L GNDD #PWR06
 U 1 1 582EA563
 P 1650 6200
-F 0 "#PWR07" H 1650 5950 50  0001 C CNN
+F 0 "#PWR06" H 1650 5950 50  0001 C CNN
 F 1 "GNDD" V 1655 6072 50  0000 R CNN
 F 2 "" H 1650 6200 50  0000 C CNN
@@
 $EndComp
 $Comp
-L GNDD #PWR08
+L GNDD #PWR07
 U 1 1 582F6F93
 P 2100 7300
-F 0 "#PWR08" H 2100 7050 50  0001 C CNN
+F 0 "#PWR07" H 2100 7050 50  0001 C CNN
 F 1 "GNDD" V 2100 7050 50  0000 C CNN
 F 2 "" H 2100 7300 50  0000 C CNN
@@
 $EndComp
 $Comp
-L VDD #PWR09
+L VDD #PWR08
 U 1 1 582F7FA8
 P 2200 7300
-F 0 "#PWR09" H 2200 7150 50  0001 C CNN
+F 0 "#PWR08" H 2200 7150 50  0001 C CNN
 F 1 "VDD" V 2200 7500 50  0000 C CNN
 F 2 "" H 2200 7300 50  0000 C CNN
@@
 $EndComp
 $Comp
-L VDD #PWR010
+L VDD #PWR09
 U 1 1 582F87A4
 P 2000 7300
-F 0 "#PWR010" H 2000 7150 50  0001 C CNN
+F 0 "#PWR09" H 2000 7150 50  0001 C CNN
 F 1 "VDD" V 2000 7500 50  0000 C CNN
 F 2 "" H 2000 7300 50  0000 C CNN
@@
 $EndComp
 $Comp
-L VDD #PWR011
+L VDD #PWR010
 U 1 1 582F88B7
 P 1900 7300
-F 0 "#PWR011" H 1900 7150 50  0001 C CNN
+F 0 "#PWR010" H 1900 7150 50  0001 C CNN
 F 1 "VDD" V 1900 7500 50  0000 C CNN
 F 2 "" H 1900 7300 50  0000 C CNN
@@
 $EndComp
 $Comp
-L GNDD #PWR012
+L GNDD #PWR011
 U 1 1 582FC419
 P 2200 5650
-F 0 "#PWR012" H 2200 5400 50  0001 C CNN
+F 0 "#PWR011" H 2200 5400 50  0001 C CNN
 F 1 "GNDD" V 2200 5400 50  0000 C CNN
 F 2 "" H 2200 5650 50  0000 C CNN
@@
 $EndComp
 $Comp
-L GNDD #PWR013
+L GNDD #PWR012
 U 1 1 582FC718
 P 1950 5650
-F 0 "#PWR013" H 1950 5400 50  0001 C CNN
+F 0 "#PWR012" H 1950 5400 50  0001 C CNN
 F 1 "GNDD" V 1950 5400 50  0000 C CNN
 F 2 "" H 1950 5650 50  0000 C CNN
@@
 $EndComp
 $Comp
-L GNDD #PWR014
+L GNDD #PWR013
 U 1 1 58310A6A
 P 5400 3250
-F 0 "#PWR014" H 5400 3000 50  0001 C CNN
+F 0 "#PWR013" H 5400 3000 50  0001 C CNN
 F 1 "GNDD" H 5400 3100 50  0000 C CNN
 F 2 "" H 5400 3250 50  0000 C CNN
@@
 $EndComp
 $Comp
-L GNDD #PWR015
+L GNDD #PWR014
 U 1 1 58311616
 P 4800 4150
-F 0 "#PWR015" H 4800 3900 50  0001 C CNN
+F 0 "#PWR014" H 4800 3900 50  0001 C CNN
 F 1 "GNDD" H 4800 4000 50  0000 C CNN
 F 2 "" H 4800 4150 50  0000 C CNN
@@
 $EndComp
 $Comp
-L VDD #PWR016
+L VDD #PWR015
 U 1 1 5831B08E
 P 4800 1050
-F 0 "#PWR016" H 4800 900 50  0001 C CNN
+F 0 "#PWR015" H 4800 900 50  0001 C CNN
 F 1 "VDD" H 4800 1200 50  0000 C CNN
 F 2 "" H 4800 1050 50  0000 C CNN
@@
 $EndComp
 $Comp
-L GNDD #PWR017
+L GNDD #PWR016
 U 1 1 5831B0B3
 P 5400 1050
-F 0 "#PWR017" H 5400 800 50  0001 C CNN
+F 0 "#PWR016" H 5400 800 50  0001 C CNN
 F 1 "GNDD" H 5400 900 50  0000 C CNN
 F 2 "" H 5400 1050 50  0000 C CNN
@@
 $EndComp
 $Comp
-L GNDD #PWR018
+L GNDD #PWR017
 U 1 1 5831B0B9
 P 4800 1950
-F 0 "#PWR018" H 4800 1700 50  0001 C CNN
+F 0 "#PWR017" H 4800 1700 50  0001 C CNN
 F 1 "GNDD" H 4800 1800 50  0000 C CNN
 F 2 "" H 4800 1950 50  0000 C CNN
@@
 BTN_OPEN
 $Comp
-L VDD #PWR019
+L VDD #PWR018
 U 1 1 5835543A
 P 5500 5950
-F 0 "#PWR019" H 5500 5800 50  0001 C CNN
+F 0 "#PWR018" H 5500 5800 50  0001 C CNN
 F 1 "VDD" V 5500 6150 50  0000 C CNN
 F 2 "" H 5500 5950 50  0000 C CNN
@@
 $EndComp
 $Comp
-L GNDD #PWR020
+L GNDD #PWR019
 U 1 1 58355464
 P 4900 6150
-F 0 "#PWR020" H 4900 5900 50  0001 C CNN
+F 0 "#PWR019" H 4900 5900 50  0001 C CNN
 F 1 "GNDD" V 4905 6022 50  0000 R CNN
 F 2 "" H 4900 6150 50  0000 C CNN
@@
 $EndComp
 $Comp
-L GNDD #PWR021
+L GNDD #PWR020
 U 1 1 58355470
 P 5350 7250
-F 0 "#PWR021" H 5350 7000 50  0001 C CNN
+F 0 "#PWR020" H 5350 7000 50  0001 C CNN
 F 1 "GNDD" V 5350 7000 50  0000 C CNN
 F 2 "" H 5350 7250 50  0000 C CNN
@@
 $EndComp
 $Comp
-L VDD #PWR022
+L VDD #PWR021
 U 1 1 58355476
 P 5450 7250
-F 0 "#PWR022" H 5450 7100 50  0001 C CNN
+F 0 "#PWR021" H 5450 7100 50  0001 C CNN
 F 1 "VDD" V 5450 7450 50  0000 C CNN
 F 2 "" H 5450 7250 50  0000 C CNN
@@
 $EndComp
 $Comp
-L VDD #PWR023
+L VDD #PWR022
 U 1 1 5835547C
 P 5250 7250
-F 0 "#PWR023" H 5250 7100 50  0001 C CNN
+F 0 "#PWR022" H 5250 7100 50  0001 C CNN
 F 1 "VDD" V 5250 7450 50  0000 C CNN
 F 2 "" H 5250 7250 50  0000 C CNN
@@
 $EndComp
 $Comp
-L VDD #PWR024
+L VDD #PWR023
 U 1 1 58355482
 P 5150 7250
-F 0 "#PWR024" H 5150 7100 50  0001 C CNN
+F 0 "#PWR023" H 5150 7100 50  0001 C CNN
 F 1 "VDD" V 5150 7450 50  0000 C CNN
 F 2 "" H 5150 7250 50  0000 C CNN
@@
 $EndComp
 $Comp
-L GNDD #PWR025
+L GNDD #PWR024
 U 1 1 58355488
 P 5450 5600
-F 0 "#PWR025" H 5450 5350 50  0001 C CNN
+F 0 "#PWR024" H 5450 5350 50  0001 C CNN
 F 1 "GNDD" V 5450 5350 50  0000 C CNN
 F 2 "" H 5450 5600 50  0000 C CNN
@@
 $EndComp
 $Comp
-L GNDD #PWR026
+L GNDD #PWR025
 U 1 1 5835548E
 P 5200 5600
-F 0 "#PWR026" H 5200 5350 50  0001 C CNN
+F 0 "#PWR025" H 5200 5350 50  0001 C CNN
 F 1 "GNDD" V 5200 5350 50  0000 C CNN
 F 2 "" H 5200 5600 50  0000 C CNN
@@
 RCCA
 $Comp
-L GNDD #PWR027
+L GNDD #PWR026
 U 1 1 583814D2
 P 9350 5450
-F 0 "#PWR027" H 9350 5200 50  0001 C CNN
+F 0 "#PWR026" H 9350 5200 50  0001 C CNN
 F 1 "GNDD" H 9350 5300 50  0000 C CNN
 F 2 "" H 9350 5450 50  0000 C CNN
@@
 $EndComp
 $Comp
-L GNDD #PWR028
+L GNDD #PWR027
 U 1 1 58381774
 P 8450 6100
-F 0 "#PWR028" H 8450 5850 50  0001 C CNN
+F 0 "#PWR027" H 8450 5850 50  0001 C CNN
 F 1 "GNDD" V 8450 5850 50  0000 C CNN
 F 2 "" H 8450 6100 50  0000 C CNN
@@
 $EndComp
 $Comp
-L GNDD #PWR029
+L GNDD #PWR028
 U 1 1 583AE5EE
 P 9100 5450
-F 0 "#PWR029" H 9100 5200 50  0001 C CNN
+F 0 "#PWR028" H 9100 5200 50  0001 C CNN
 F 1 "GNDD" H 9100 5300 50  0000 C CNN
 F 2 "" H 9100 5450 50  0000 C CNN
@@
 $EndComp
 $Comp
-L VDD #PWR030
+L VDD #PWR029
 U 1 1 583B6020
 P 9450 6000
-F 0 "#PWR030" H 9450 5850 50  0001 C CNN
+F 0 "#PWR029" H 9450 5850 50  0001 C CNN
 F 1 "VDD" V 9450 6200 50  0000 C CNN
 F 2 "" H 9450 6000 50  0000 C CNN
@@
 Connection ~ 2800 1050
 $Comp
-L VDD #PWR031
+L VDD #PWR030
 U 1 1 58223ACA
 P 3150 1050
-F 0 "#PWR031" H 3150 900 50  0001 C CNN
+F 0 "#PWR030" H 3150 900 50  0001 C CNN
 F 1 "VDD" V 3150 1250 50  0000 C CNN
 F 2 "" H 3150 1050 50  0000 C CNN
@@
 $EndComp
 $Comp
-L VDD #PWR032
+L VDD #PWR031
 U 1 1 582264A1
 P 3150 1250
-F 0 "#PWR032" H 3150 1100 50  0001 C CNN
+F 0 "#PWR031" H 3150 1100 50  0001 C CNN
 F 1 "VDD" V 3150 1450 50  0000 C CNN
 F 2 "" H 3150 1250 50  0000 C CNN
@@
 Wire Wire Line
 	8850 3250 8950 3250
+$Comp
+L GNDPWR #PWR032
+U 1 1 58586DF6
+P 8850 4450
+F 0 "#PWR032" H 8850 4250 50  0001 C CNN
+F 1 "GNDPWR" H 8850 4275 50  0000 C CNN
+F 2 "" H 8850 4400 50  0000 C CNN
+F 3 "" H 8850 4400 50  0000 C CNN
+	1    8850 4450
+	1    0    0    -1
+$EndComp
 $EndSCHEMATC

Commit message: fix PCB problems
Parts:
- added R29, R30, R31: 4.7k, I20:R_0805, symbol R
- R22: value 0 -> 4.7k
Connections:
- net ESP_RESET: now also R31.2
- net VDD: now also R29.2, R30.2, R31.1
- net at P6.3 (P3): now also R29.1
- net at P6.5 (P5): now also R30.1
- no-connect marks 4 -> 2

Commit message: align with recent develop changes
Parts:
- removed Q4: Q_NMOS_DGS, I20:SOT-23, symbol Q_NMOS_DGS
- added Q4: MOSFET-NCHANNELSMD, SparkFun-SOT23-3, symbol MOSFET-NCHANNELSMD
Connections:
- net GNDPWR: now also Q4.2 (S)
- net LOCK_GND: now also Q4.3 (D)
- net at D3.1 (K), R23.1, R24.2: now also Q4.1 (G)
Changed lines of the file:
@@
 EESchema Schematic File Version 2
-LIBS:em-lock-rescue
 LIBS:power
 LIBS:device
@@
 $EndComp
 $Comp
-L VDD #PWR2
+L VDD #PWR01
 U 1 1 57BF1F35
 P 1700 3000
-F 0 "#PWR2" H 1700 2850 50  0001 C CNN
+F 0 "#PWR01" H 1700 2850 50  0001 C CNN
 F 1 "VDD" H 1717 3173 50  0000 C CNN
 F 2 "" H 1700 3000 50  0000 C CNN
@@
 $EndComp
 $Comp
-L VDD #PWR33
+L VDD #PWR02
 U 1 1 57BFC190
 P 9450 5800
-F 0 "#PWR33" H 9450 5650 50  0001 C CNN
+F 0 "#PWR02" H 9450 5650 50  0001 C CNN
 F 1 "VDD" V 9450 6000 50  0000 C CNN
 F 2 "" H 9450 5800 50  0000 C CNN
@@
 	1    9100 5600
 	1    0    0    -1
-$EndComp
-$Comp
-L Q_NMOS_DGS Q4
-U 1 1 57BF2360
-P 8950 3800
-F 0 "Q4" H 8800 3950 50  0000 L CNN
-F 1 "Q_NMOS_DGS" V 9200 3500 50  0000 L CNN
-F 2 "I20:SOT-23" H 9150 3900 50  0001 C CNN
-F 3 "" H 8950 3800 50  0000 C CNN
-	1    8950 3800
-	-1   0    0    -1
 $EndComp
 $Comp
@@
 $EndComp
 $Comp
-L VDD #PWR15
+L VDD #PWR03
 U 1 1 57BFAAAC
 P 4800 3250
-F 0 "#PWR15" H 4800 3100 50  0001 C CNN
+F 0 "#PWR03" H 4800 3100 50  0001 C CNN
 F 1 "VDD" H 4800 3400 50  0000 C CNN
 F 2 "" H 4800 3250 50  0000 C CNN
@@
 $EndComp
 $Comp
-L GNDD #PWR10
+L GNDD #PWR04
 U 1 1 582803A4
 P 2800 950
-F 0 "#PWR10" H 2800 700 50  0001 C CNN
+F 0 "#PWR04" H 2800 700 50  0001 C CNN
 F 1 "GNDD" H 2800 800 50  0000 C CNN
 F 2 "" H 2800 950 50  0000 C CNN
@@
 $EndComp
 $Comp
-L VDD #PWR9
+L VDD #PWR05
 U 1 1 5829C375
 P 2250 6000
-F 0 "#PWR9" H 2250 5850 50  0001 C CNN
+F 0 "#PWR05" H 2250 5850 50  0001 C CNN
 F 1 "VDD" V 2250 6200 50  0000 C CNN
 F 2 "" H 2250 6000 50  0000 C CNN
@@
 $EndComp
 $Comp
-L GNDD #PWR1
+L GNDD #PWR06
 U 1 1 582EA563
 P 1650 6200
-F 0 "#PWR1" H 1650 5950 50  0001 C CNN
+F 0 "#PWR06" H 1650 5950 50  0001 C CNN
 F 1 "GNDD" V 1655 6072 50  0000 R CNN
 F 2 "" H 1650 6200 50  0000 C CNN
@@
 $EndComp
 $Comp
-L GNDD #PWR6
+L GNDD #PWR07
 U 1 1 582F6F93
 P 2100 7300
-F 0 "#PWR6" H 2100 7050 50  0001 C CNN
+F 0 "#PWR07" H 2100 7050 50  0001 C CNN
 F 1 "GNDD" V 2100 7050 50  0000 C CNN
 F 2 "" H 2100 7300 50  0000 C CNN
@@
 $EndComp
 $Comp
-L VDD #PWR8
+L VDD #PWR08
 U 1 1 582F7FA8
 P 2200 7300
-F 0 "#PWR8" H 2200 7150 50  0001 C CNN
+F 0 "#PWR08" H 2200 7150 50  0001 C CNN
 F 1 "VDD" V 2200 7500 50  0000 C CNN
 F 2 "" H 2200 7300 50  0000 C CNN
@@
 $EndComp
 $Comp
-L VDD #PWR5
+L VDD #PWR09
 U 1 1 582F87A4
 P 2000 7300
-F 0 "#PWR5" H 2000 7150 50  0001 C CNN
+F 0 "#PWR09" H 2000 7150 50  0001 C CNN
 F 1 "VDD" V 2000 7500 50  0000 C CNN
 F 2 "" H 2000 7300 50  0000 C CNN
@@
 $EndComp
 $Comp
-L VDD #PWR3
+L VDD #PWR010
 U 1 1 582F88B7
 P 1900 7300
-F 0 "#PWR3" H 1900 7150 50  0001 C CNN
+F 0 "#PWR010" H 1900 7150 50  0001 C CNN
 F 1 "VDD" V 1900 7500 50  0000 C CNN
 F 2 "" H 1900 7300 50  0000 C CNN
@@
 $EndComp
 $Comp
-L GNDD #PWR7
+L GNDD #PWR011
 U 1 1 582FC419
 P 2200 5650
-F 0 "#PWR7" H 2200 5400 50  0001 C CNN
+F 0 "#PWR011" H 2200 5400 50  0001 C CNN
 F 1 "GNDD" V 2200 5400 50  0000 C CNN
 F 2 "" H 2200 5650 50  0000 C CNN
@@
 $EndComp
 $Comp
-L GNDD #PWR4
+L GNDD #PWR012
 U 1 1 582FC718
 P 1950 5650
-F 0 "#PWR4" H 1950 5400 50  0001 C CNN
+F 0 "#PWR012" H 1950 5400 50  0001 C CNN
 F 1 "GNDD" V 1950 5400 50  0000 C CNN
 F 2 "" H 1950 5650 50  0000 C CNN
@@
 $EndComp
 $Comp
-L GNDD #PWR23
+L GNDD #PWR013
 U 1 1 58310A6A
 P 5400 3250
-F 0 "#PWR23" H 5400 3000 50  0001 C CNN
+F 0 "#PWR013" H 5400 3000 50  0001 C CNN
 F 1 "GNDD" H 5400 3100 50  0000 C CNN
 F 2 "" H 5400 3250 50  0000 C CNN
@@
 $EndComp
 $Comp
-L GNDD #PWR16
+L GNDD #PWR014
 U 1 1 58311616
 P 4800 4150
-F 0 "#PWR16" H 4800 3900 50  0001 C CNN
+F 0 "#PWR014" H 4800 3900 50  0001 C CNN
 F 1 "GNDD" H 4800 4000 50  0000 C CNN
 F 2 "" H 4800 4150 50  0000 C CNN
@@
 $EndComp
 $Comp
-L VDD #PWR13
+L VDD #PWR015
 U 1 1 5831B08E
 P 4800 1050
-F 0 "#PWR13" H 4800 900 50  0001 C CNN
+F 0 "#PWR015" H 4800 900 50  0001 C CNN
 F 1 "VDD" H 4800 1200 50  0000 C CNN
 F 2 "" H 4800 1050 50  0000 C CNN
@@
 $EndComp
 $Comp
-L GNDD #PWR22
+L GNDD #PWR016
 U 1 1 5831B0B3
 P 5400 1050
-F 0 "#PWR22" H 5400 800 50  0001 C CNN
+F 0 "#PWR016" H 5400 800 50  0001 C CNN
 F 1 "GNDD" H 5400 900 50  0000 C CNN
 F 2 "" H 5400 1050 50  0000 C CNN
@@
 $EndComp
 $Comp
-L GNDD #PWR14
+L GNDD #PWR017
 U 1 1 5831B0B9
 P 4800 1950
-F 0 "#PWR14" H 4800 1700 50  0001 C CNN
+F 0 "#PWR017" H 4800 1700 50  0001 C CNN
 F 1 "GNDD" H 4800 1800 50  0000 C CNN
 F 2 "" H 4800 1950 50  0000 C CNN
@@
 BTN_OPEN
 $Comp
-L VDD #PWR26
+L VDD #PWR018
 U 1 1 5835543A
 P 5500 5950
-F 0 "#PWR26" H 5500 5800 50  0001 C CNN
+F 0 "#PWR018" H 5500 5800 50  0001 C CNN
 F 1 "VDD" V 5500 6150 50  0000 C CNN
 F 2 "" H 5500 5950 50  0000 C CNN
@@
 $EndComp
 $Comp
-L GNDD #PWR17
+L GNDD #PWR019
 U 1 1 58355464
 P 4900 6150
-F 0 "#PWR17" H 4900 5900 50  0001 C CNN
+F 0 "#PWR019" H 4900 5900 50  0001 C CNN
 F 1 "GNDD" V 4905 6022 50  0000 R CNN
 F 2 "" H 4900 6150 50  0000 C CNN
@@
 $EndComp
 $Comp
-L GNDD #PWR21
+L GNDD #PWR020
 U 1 1 58355470
 P 5350 7250
-F 0 "#PWR21" H 5350 7000 50  0001 C CNN
+F 0 "#PWR020" H 5350 7000 50  0001 C CNN
 F 1 "GNDD" V 5350 7000 50  0000 C CNN
 F 2 "" H 5350 7250 50  0000 C CNN
@@
 $EndComp
 $Comp
-L VDD #PWR25
+L VDD #PWR021
 U 1 1 58355476
 P 5450 7250
-F 0 "#PWR25" H 5450 7100 50  0001 C CNN
+F 0 "#PWR021" H 5450 7100 50  0001 C CNN
 F 1 "VDD" V 5450 7450 50  0000 C CNN
 F 2 "" H 5450 7250 50  0000 C CNN
@@
 $EndComp
 $Comp
-L VDD #PWR20
+L VDD #PWR022
 U 1 1 5835547C
 P 5250 7250
-F 0 "#PWR20" H 5250 7100 50  0001 C CNN
+F 0 "#PWR022" H 5250 7100 50  0001 C CNN
 F 1 "VDD" V 5250 7450 50  0000 C CNN
 F 2 "" H 5250 7250 50  0000 C CNN
@@
 $EndComp
 $Comp
-L VDD #PWR18
+L VDD #PWR023
 U 1 1 58355482
 P 5150 7250
-F 0 "#PWR18" H 5150 7100 50  0001 C CNN
+F 0 "#PWR023" H 5150 7100 50  0001 C CNN
 F 1 "VDD" V 5150 7450 50  0000 C CNN
 F 2 "" H 5150 7250 50  0000 C CNN
@@
 $EndComp
 $Comp
-L GNDD #PWR24
+L GNDD #PWR024
 U 1 1 58355488
 P 5450 5600
-F 0 "#PWR24" H 5450 5350 50  0001 C CNN
+F 0 "#PWR024" H 5450 5350 50  0001 C CNN
 F 1 "GNDD" V 5450 5350 50  0000 C CNN
 F 2 "" H 5450 5600 50  0000 C CNN
@@
 $EndComp
 $Comp
-L GNDD #PWR19
+L GNDD #PWR025
 U 1 1 5835548E
 P 5200 5600
-F 0 "#PWR19" H 5200 5350 50  0001 C CNN
+F 0 "#PWR025" H 5200 5350 50  0001 C CNN
 F 1 "GNDD" V 5200 5350 50  0000 C CNN
 F 2 "" H 5200 5600 50  0000 C CNN
@@
 RCCA
 $Comp
-L GNDD #PWR32
+L GNDD #PWR026
 U 1 1 583814D2
 P 9350 5450
-F 0 "#PWR32" H 9350 5200 50  0001 C CNN
+F 0 "#PWR026" H 9350 5200 50  0001 C CNN
 F 1 "GNDD" H 9350 5300 50  0000 C CNN
 F 2 "" H 9350 5450 50  0000 C CNN
@@
 $EndComp
 $Comp
-L GNDD #PWR29
+L GNDD #PWR027
 U 1 1 58381774
 P 8125 6100
-F 0 "#PWR29" H 8125 5850 50  0001 C CNN
+F 0 "#PWR027" H 8125 5850 50  0001 C CNN
 F 1 "GNDD" V 8125 5850 50  0000 C CNN
 F 2 "" H 8125 6100 50  0000 C CNN
@@
 $EndComp
 $Comp
-L GNDD #PWR31
+L GNDD #PWR028
 U 1 1 583AE5EE
 P 9100 5450
-F 0 "#PWR31" H 9100 5200 50  0001 C CNN
+F 0 "#PWR028" H 9100 5200 50  0001 C CNN
 F 1 "GNDD" H 9100 5300 50  0000 C CNN
 F 2 "" H 9100 5450 50  0000 C CNN
@@
 $EndComp
 $Comp
-L VDD #PWR34
+L VDD #PWR029
 U 1 1 583B6020
 P 9450 6000
-F 0 "#PWR34" H 9450 5850 50  0001 C CNN
+F 0 "#PWR029" H 9450 5850 50  0001 C CNN
 F 1 "VDD" V 9450 6200 50  0000 C CNN
 F 2 "" H 9450 6000 50  0000 C CNN
@@
 $EndComp
 $Comp
-L VDD #PWR11
+L VDD #PWR030
 U 1 1 58223ACA
 P 3150 1050
-F 0 "#PWR11" H 3150 900 50  0001 C CNN
+F 0 "#PWR030" H 3150 900 50  0001 C CNN
 F 1 "VDD" V 3150 1250 50  0000 C CNN
 F 2 "" H 3150 1050 50  0000 C CNN
@@
 $EndComp
 $Comp
-L VDD #PWR12
+L VDD #PWR031
 U 1 1 582264A1
 P 3150 1250
-F 0 "#PWR12" H 3150 1100 50  0001 C CNN
+F 0 "#PWR031" H 3150 1100 50  0001 C CNN
 F 1 "VDD" V 3150 1450 50  0000 C CNN
 F 2 "" H 3150 1250 50  0000 C CNN
@@
 EM_LOCK
 $Comp
-L GNDPWR #PWR30
+L GNDPWR #PWR032
 U 1 1 58586DF6
 P 8850 4450
-F 0 "#PWR30" H 8850 4250 50  0001 C CNN
+F 0 "#PWR032" H 8850 4250 50  0001 C CNN
 F 1 "GNDPWR" H 8850 4275 50  0000 C CNN
 F 2 "" H 8850 4400 50  0000 C CNN
@@
 $EndComp
 $Comp
-L VDD #PWR28
+L VDD #PWR033
 U 1 1 58718815
 P 8125 6000
-F 0 "#PWR28" H 8125 5850 50  0001 C CNN
+F 0 "#PWR033" H 8125 5850 50  0001 C CNN
 F 1 "VDD" V 8125 6200 50  0000 C CNN
 F 2 "" H 8125 6000 50  0000 C CNN
@@
 $EndComp
 $Comp
-L VDD #PWR27
+L VDD #PWR034
 U 1 1 5871B4C1
 P 8125 5900
-F 0 "#PWR27" H 8125 5750 50  0001 C CNN
+F 0 "#PWR034" H 8125 5750 50  0001 C CNN
 F 1 "VDD" V 8125 6100 50  0000 C CNN
 F 2 "" H 8125 5900 50  0000 C CNN
@@
 $EndComp
 $Comp
-L VDD #PWR35
+L VDD #PWR035
 U 1 1 58729F36
 P 9750 5450
-F 0 "#PWR35" H 9750 5300 50  0001 C CNN
+F 0 "#PWR035" H 9750 5300 50  0001 C CNN
 F 1 "VDD" H 9750 5600 50  0000 C CNN
 F 2 "" H 9750 5450 50  0000 C CNN
@@
 Wire Wire Line
 	9500 4300 9500 4250
-Connection ~ 8850 4300
 Wire Wire Line
 	8850 4300 9500 4300
-Connection ~ 9150 3800
 Wire Wire Line
 	9150 3850 9150 3800
@@
 Wire Wire Line
 	9000 5900 9850 5900
+$Comp
+L MOSFET-NCHANNELSMD Q4
+U 1 1 58A34D60
+P 8850 3800
+F 0 "Q4" H 9013 3754 50  0000 L CNN
+F 1 "MOSFET-NCHANNELSMD" V 9300 3200 50  0000 L CNN
+F 2 "SparkFun-SOT23-3" H 9400 3800 50  0001 C CNN
+F 3 "" H 8850 3800 60  0001 C CNN
+	1    8850 3800
+	-1   0    0    -1
+$EndComp
+Connection ~ 8850 4300
+Connection ~ 9150 3800
+Connection ~ 4700 6200
+Connection ~ 8850 3600
+Connection ~ 8850 4000
 $EndSCHEMATC
