File: eda/stm32.sch (KiCad schematic (older format))
At the start: 27 parts, among them CON1 BARREL_JACK, P10 BOOT_SEL_CONN, P12 SWD_CONN, P9 PWR_SW_CONN, SW1 RST_BTN, U2 LD1117S33CTR, U3 STM32F103C8Tx, Y1 8MHz

Commit message: fix PCB before manufacturing
Connections:
- net GNDREF is gone; now on net GNDD: C10.2, C11.2, C12.2, C13.1, C16.2, C17.2, C18.2, C19.1, C20.1, C9.2, CON1.2, CON1.3, D4.2 (A), P12.4 (P4), SW1.1, U2.1 (GND), U3.23 (VSS), U3.35 (VSS), U3.47 (VSS), U3.8 (VSSA)
- net GNDD: now reaches C14.2, C15.2
- net GNDD: now also P10.5 (P5), P10.6 (P6)
Changed lines of the file:
@@
 EESchema Schematic File Version 2
+LIBS:em-lock-rescue
 LIBS:power
 LIBS:device
@@
 $EndComp
 $Comp
-L GND #PWR034
+L GNDD #PWR034
 U 1 1 57BED7A6
 P 2000 1900
+AR Path="/57BED7A6" Ref="#PWR034"  Part="1"
+AR Path="/5818E6EE/57BED7A6" Ref="#PWR034"  Part="1"
 F 0 "#PWR034" H 2000 1650 50  0001 C CNN
-F 1 "GND" H 2005 1727 50  0000 C CNN
+F 1 "GNDD" H 2005 1727 50  0000 C CNN
 F 2 "" H 2000 1900 50  0000 C CNN
 F 3 "" H 2000 1900 50  0000 C CNN
@@
 $EndComp
 $Comp
-L GND #PWR035
+L GNDREF #PWR035
 U 1 1 581973BA
 P 11200 7400
+AR Path="/581973BA" Ref="#PWR035"  Part="1"
+AR Path="/5818E6EE/581973BA" Ref="#PWR035"  Part="1"
 F 0 "#PWR035" H 11200 7150 50  0001 C CNN
-F 1 "GND" H 11205 7227 50  0000 C CNN
+F 1 "GNDREF" H 11205 7227 50  0000 C CNN
 F 2 "" H 11200 7400 50  0000 C CNN
 F 3 "" H 11200 7400 50  0000 C CNN
@@
 $EndComp
 $Comp
-L GND #PWR037
+L GNDD #PWR037
 U 1 1 581973C9
 P 6150 2250
+AR Path="/581973C9" Ref="#PWR037"  Part="1"
+AR Path="/5818E6EE/581973C9" Ref="#PWR037"  Part="1"
 F 0 "#PWR037" H 6150 2000 50  0001 C CNN
-F 1 "GND" H 6155 2077 50  0000 C CNN
+F 1 "GNDD" H 6155 2077 50  0000 C CNN
 F 2 "" H 6150 2250 50  0000 C CNN
 F 3 "" H 6150 2250 50  0000 C CNN
@@
 F 3 "" H 4400 5050 50  0000 C CNN
 	1    4400 5050
-	1    0    0    -1
-$EndComp
-$Comp
-L GND #PWR039
-U 1 1 581973CC
-P 4400 5550
-F 0 "#PWR039" H 4400 5300 50  0001 C CNN
-F 1 "GND" H 4405 5377 50  0000 C CNN
-F 2 "" H 4400 5550 50  0000 C CNN
-F 3 "" H 4400 5550 50  0000 C CNN
-	1    4400 5550
 	1    0    0    -1
 $EndComp
@@
 $EndComp
 $Comp
-L GND #PWR040
+L GNDREF #PWR040
 U 1 1 581973D5
 P 4400 4000
-F 0 "#PWR040" H 4400 3750 50  0001 C CNN
-F 1 "GND" V 4300 3800 50  0000 C CNN
+AR Path="/581973D5" Ref="#PWR040"  Part="1"
+AR Path="/5818E6EE/581973D5" Ref="#PWR039"  Part="1"
+F 0 "#PWR039" H 4400 3750 50  0001 C CNN
+F 1 "GNDREF" H 4300 3825 50  0000 C CNN
 F 2 "" H 4400 4000 50  0000 C CNN
 F 3 "" H 4400 4000 50  0000 C CNN
@@
 $EndComp
 $Comp
-L GND #PWR041
+L GNDREF #PWR041
 U 1 1 581BD405
 P 9950 9590
-F 0 "#PWR041" H 9950 9340 50  0001 C CNN
-F 1 "GND" H 9955 9417 50  0000 C CNN
+AR Path="/581BD405" Ref="#PWR041"  Part="1"
+AR Path="/5818E6EE/581BD405" Ref="#PWR040"  Part="1"
+F 0 "#PWR040" H 9950 9340 50  0001 C CNN
+F 1 "GNDREF" H 10040 9415 50  0000 C CNN
 F 2 "" H 9950 9590 50  0000 C CNN
 F 3 "" H 9950 9590 50  0000 C CNN
@@
 $EndComp
 $Comp
-L VDD #PWR042
+L VDD #PWR041
 U 1 1 581BD6DF
 P 9950 9890
-F 0 "#PWR042" H 9950 9740 50  0001 C CNN
+F 0 "#PWR041" H 9950 9740 50  0001 C CNN
 F 1 "VDD" H 9967 10063 50  0000 C CNN
 F 2 "" H 9950 9890 50  0000 C CNN
@@
 $EndComp
 $Comp
-L VCC #PWR043
+L VCC #PWR042
 U 1 1 581973DA
 P 5250 4750
-F 0 "#PWR043" H 5250 4600 50  0001 C CNN
+F 0 "#PWR042" H 5250 4600 50  0001 C CNN
 F 1 "VCC" H 5267 4923 50  0000 C CNN
 F 2 "" H 5250 4750 50  0000 C CNN
@@
 $EndComp
 $Comp
-L VDD #PWR044
+L VDD #PWR043
 U 1 1 57BEF7FC
 P 5050 4750
-F 0 "#PWR044" H 5050 4600 50  0001 C CNN
+F 0 "#PWR043" H 5050 4600 50  0001 C CNN
 F 1 "VDD" H 5067 4923 50  0000 C CNN
 F 2 "" H 5050 4750 50  0000 C CNN
@@
 SWCLK
 $Comp
-L GND #PWR045
+L GNDD #PWR045
 U 1 1 57BDD879
 P 12400 4450
-F 0 "#PWR045" H 12400 4200 50  0001 C CNN
-F 1 "GND" H 12405 4277 50  0000 C CNN
+AR Path="/57BDD879" Ref="#PWR045"  Part="1"
+AR Path="/5818E6EE/57BDD879" Ref="#PWR044"  Part="1"
+F 0 "#PWR044" H 12400 4200 50  0001 C CNN
+F 1 "GNDD" H 12405 4277 50  0000 C CNN
 F 2 "" H 12400 4450 50  0000 C CNN
 F 3 "" H 12400 4450 50  0000 C CNN
@@
 Wire Wire Line
 	3750 3950 3750 4100
+$Comp
+L GNDPWR #PWR045
+U 1 1 58599527
+P 4400 5550
+F 0 "#PWR045" H 4400 5350 50  0001 C CNN
+F 1 "GNDPWR" H 4100 5500 50  0000 C CNN
+F 2 "" H 4400 5500 50  0000 C CNN
+F 3 "" H 4400 5500 50  0000 C CNN
+	1    4400 5550
+	1    0    0    -1
+$EndComp
+Connection ~ 6150 2250
+Connection ~ 11200 7400
+$Comp
+L GNDPWR #PWR046
+U 1 1 5859FEF8
+P 1775 4075
+F 0 "#PWR046" H 1775 3875 50  0001 C CNN
+F 1 "GNDPWR" H 1475 4025 50  0000 C CNN
+F 2 "" H 1775 4025 50  0000 C CNN
+F 3 "" H 1775 4025 50  0000 C CNN
+	1    1775 4075
+	-1   0    0    1
+$EndComp
+$Comp
+L GNDD #PWR047
+U 1 1 585A01F7
+P 1600 4075
+F 0 "#PWR047" H 1600 3825 50  0001 C CNN
+F 1 "GNDD" H 1800 4025 50  0000 C CNN
+F 2 "" H 1600 4075 50  0000 C CNN
+F 3 "" H 1600 4075 50  0000 C CNN
+	1    1600 4075
+	-1   0    0    1
+$EndComp
+$Comp
+L GNDREF #PWR048
+U 1 1 585A0562
+P 1700 4225
+F 0 "#PWR048" H 1700 3975 50  0001 C CNN
+F 1 "GNDREF" H 1705 4052 50  0000 C CNN
+F 2 "" H 1700 4225 50  0000 C CNN
+F 3 "" H 1700 4225 50  0000 C CNN
+	1    1700 4225
+	1    0    0    -1
+$EndComp
+Wire Wire Line
+	1600 4075 1600 4150
+Wire Wire Line
+	1600 4150 1775 4150
+Wire Wire Line
+	1700 4150 1700 4225
+Wire Wire Line
+	1775 4150 1775 4075
+Connection ~ 1700 4150
 $EndSCHEMATC

Commit message: align with recent develop changes
Connections:
- net VCC: now also P10.1 (P1), P10.2 (P2)
Changed lines of the file:
@@
 EESchema Schematic File Version 2
-LIBS:em-lock-rescue
 LIBS:power
 LIBS:device
@@
 $EndDescr
 $Comp
-L VDD #PWR50
+L VDD #PWR036
 U 1 1 57BED091
 P 12050 750
-F 0 "#PWR50" H 12050 600 50  0001 C CNN
+F 0 "#PWR036" H 12050 600 50  0001 C CNN
 F 1 "VDD" V 12100 700 50  0000 C CNN
 F 2 "" H 12050 750 50  0000 C CNN
@@
 P 2000 1900
 AR Path="/57BED7A6" Ref="#PWR034"  Part="1"
-AR Path="/5818E6EE/57BED7A6" Ref="#PWR39"  Part="1"
-F 0 "#PWR39" H 2000 1650 50  0001 C CNN
+AR Path="/5818E6EE/57BED7A6" Ref="#PWR037"  Part="1"
+F 0 "#PWR037" H 2000 1650 50  0001 C CNN
 F 1 "GNDD" H 2005 1727 50  0000 C CNN
 F 2 "" H 2000 1900 50  0000 C CNN
@@
 P 11200 7400
 AR Path="/581973BA" Ref="#PWR035"  Part="1"
-AR Path="/5818E6EE/581973BA" Ref="#PWR49"  Part="1"
-F 0 "#PWR49" H 11200 7150 50  0001 C CNN
+AR Path="/5818E6EE/581973BA" Ref="#PWR038"  Part="1"
+F 0 "#PWR038" H 11200 7150 50  0001 C CNN
 F 1 "GNDREF" H 11205 7227 50  0000 C CNN
 F 2 "" H 11200 7400 50  0000 C CNN
@@
 $EndComp
 $Comp
-L VDD #PWR40
+L VDD #PWR039
 U 1 1 581973C3
 P 2700 2300
-F 0 "#PWR40" H 2700 2150 50  0001 C CNN
+F 0 "#PWR039" H 2700 2150 50  0001 C CNN
 F 1 "VDD" H 2717 2473 50  0000 C CNN
 F 2 "" H 2700 2300 50  0000 C CNN
@@
 P 6150 2250
 AR Path="/581973C9" Ref="#PWR037"  Part="1"
-AR Path="/5818E6EE/581973C9" Ref="#PWR46"  Part="1"
-F 0 "#PWR46" H 6150 2000 50  0001 C CNN
+AR Path="/5818E6EE/581973C9" Ref="#PWR040"  Part="1"
+F 0 "#PWR040" H 6150 2000 50  0001 C CNN
 F 1 "GNDD" H 6155 2077 50  0000 C CNN
 F 2 "" H 6150 2250 50  0000 C CNN
@@
 $EndComp
 $Comp
-L VDD #PWR45
+L VDD #PWR041
 U 1 1 581973CA
 P 6150 1550
-F 0 "#PWR45" H 6150 1400 50  0001 C CNN
+F 0 "#PWR041" H 6150 1400 50  0001 C CNN
 F 1 "VDD" H 6167 1723 50  0000 C CNN
 F 2 "" H 6150 1550 50  0000 C CNN
@@
 P 4400 4000
 AR Path="/581973D5" Ref="#PWR040"  Part="1"
-AR Path="/5818E6EE/581973D5" Ref="#PWR41"  Part="1"
-F 0 "#PWR41" H 4400 3750 50  0001 C CNN
+AR Path="/5818E6EE/581973D5" Ref="#PWR042"  Part="1"
+F 0 "#PWR042" H 4400 3750 50  0001 C CNN
 F 1 "GNDREF" H 4300 3825 50  0000 C CNN
 F 2 "" H 4400 4000 50  0000 C CNN
@@
 P 9950 9590
 AR Path="/581BD405" Ref="#PWR041"  Part="1"
-AR Path="/5818E6EE/581BD405" Ref="#PWR47"  Part="1"
-F 0 "#PWR47" H 9950 9340 50  0001 C CNN
+AR Path="/5818E6EE/581BD405" Ref="#PWR043"  Part="1"
+F 0 "#PWR043" H 9950 9340 50  0001 C CNN
 F 1 "GNDREF" H 10040 9415 50  0000 C CNN
 F 2 "" H 9950 9590 50  0000 C CNN
@@
 $EndComp
 $Comp
-L VDD #PWR48
+L VDD #PWR044
 U 1 1 581BD6DF
 P 9950 9890
-F 0 "#PWR48" H 9950 9740 50  0001 C CNN
+F 0 "#PWR044" H 9950 9740 50  0001 C CNN
 F 1 "VDD" H 9967 10063 50  0000 C CNN
 F 2 "" H 9950 9890 50  0000 C CNN
@@
 $EndComp
 $Comp
-L VCC #PWR44
+L VCC #PWR045
 U 1 1 581973DA
 P 5250 4750
-F 0 "#PWR44" H 5250 4600 50  0001 C CNN
+F 0 "#PWR045" H 5250 4600 50  0001 C CNN
 F 1 "VCC" H 5267 4923 50  0000 C CNN
 F 2 "" H 5250 4750 50  0000 C CNN
@@
 $EndComp
 $Comp
-L VDD #PWR43
+L VDD #PWR046
 U 1 1 57BEF7FC
 P 5050 4750
-F 0 "#PWR43" H 5050 4600 50  0001 C CNN
+F 0 "#PWR046" H 5050 4600 50  0001 C CNN
 F 1 "VDD" H 5067 4923 50  0000 C CNN
 F 2 "" H 5050 4750 50  0000 C CNN
@@
 P 12400 4450
 AR Path="/57BDD879" Ref="#PWR045"  Part="1"
-AR Path="/5818E6EE/57BDD879" Ref="#PWR51"  Part="1"
-F 0 "#PWR51" H 12400 4200 50  0001 C CNN
+AR Path="/5818E6EE/57BDD879" Ref="#PWR047"  Part="1"
+F 0 "#PWR047" H 12400 4200 50  0001 C CNN
 F 1 "GNDD" H 12405 4277 50  0000 C CNN
 F 2 "" H 12400 4450 50  0000 C CNN
@@
 	3750 3950 3750 4100
 $Comp
-L GNDPWR #PWR42
+L GNDPWR #PWR048
 U 1 1 58599527
 P 4400 5550
-F 0 "#PWR42" H 4400 5350 50  0001 C CNN
+F 0 "#PWR048" H 4400 5350 50  0001 C CNN
 F 1 "GNDPWR" H 4100 5500 50  0000 C CNN
 F 2 "" H 4400 5500 50  0000 C CNN
@@
 Connection ~ 11200 7400
 $Comp
-L GNDPWR #PWR38
+L GNDPWR #PWR049
 U 1 1 5859FEF8
 P 1775 4075
-F 0 "#PWR38" H 1775 3875 50  0001 C CNN
+F 0 "#PWR049" H 1775 3875 50  0001 C CNN
 F 1 "GNDPWR" H 1475 4025 50  0000 C CNN
 F 2 "" H 1775 4025 50  0000 C CNN
@@
 $EndComp
 $Comp
-L GNDD #PWR36
+L GNDD #PWR050
 U 1 1 585A01F7
 P 1600 4075
-F 0 "#PWR36" H 1600 3825 50  0001 C CNN
+F 0 "#PWR050" H 1600 3825 50  0001 C CNN
 F 1 "GNDD" H 1800 4025 50  0000 C CNN
 F 2 "" H 1600 4075 50  0000 C CNN
@@
 $EndComp
 $Comp
-L GNDREF #PWR37
+L GNDREF #PWR051
 U 1 1 585A0562
 P 1700 4225
-F 0 "#PWR37" H 1700 3975 50  0001 C CNN
+F 0 "#PWR051" H 1700 3975 50  0001 C CNN
 F 1 "GNDREF" H 1705 4052 50  0000 C CNN
 F 2 "" H 1700 4225 50  0000 C CNN
@@
 	1775 4150 1775 4075
 Connection ~ 1700 4150
+Connection ~ 6150 1550
+Connection ~ 15200 1950
 $EndSCHEMATC
